Commit message: validate physical hardware bringup

File: robot_ws/src/romo_b_description/urdf/romo_b.urdf.xacro (robot description, xacro)
@@ -72,5 +72,7 @@
   <link name="livox_frame">
     <visual>
-      <geometry><cylinder radius="0.033" length="0.065"/></geometry>
+      <!-- Mid-360 origin O is 47 mm above its bottom; its body is 60 mm tall. -->
+      <origin xyz="0 0 -0.017" rpy="0 0 0"/>
+      <geometry><cylinder radius="0.0325" length="0.060"/></geometry>
       <material name="sensor_red"/>
     </visual>

Commit message: validate lidar localization replay

File: robot_ws/src/romo_b_description/urdf/romo_b.urdf.xacro (robot description, xacro)
@@ -19,7 +19,9 @@
   <link name="base_footprint"/>
   <joint name="base_footprint_joint" type="fixed">
-    <parent link="base_footprint"/>
-    <child link="base_link"/>
-    <origin xyz="0 0 ${body_height / 2.0}" rpy="0 0 0"/>
+    <!-- base_link is the dynamic odometry child. Keeping the ground-projected
+         frame below it avoids giving base_link two TF parents. -->
+    <parent link="base_link"/>
+    <child link="base_footprint"/>
+    <origin xyz="0 0 ${-body_height / 2.0}" rpy="0 0 0"/>
   </joint>
   <link name="base_link">
